Commit message: Add tugbot test data

File: urdf/tugbot_simple.urdf (robot description, URDF)
Before this commit: robot car, 1 links, 0 joints
Links:
- added link wheel_left, mass 5.45489492215439
- added link wheel_right, mass 5.45489492215438
- link base_link: mass None -> 30.9099300932655; geometry 
Joints:
- added joint wheel_left: type continuous, parent base_link, child wheel_left, origin xyz=0 0.2175 0.195 rpy=-1.5708 0.98331 -3.1416, axis 0 0 -1
- added joint wheel_right: type continuous, parent base_link, child wheel_right, origin xyz=0 -0.2175 0.195 rpy=1.5708 0 -3.1416, axis 0 0 1
